Commit message: Add rviz launches and fix direction of left motors

File: upmoon_description/urdf/upmoon_description.urdf (robot description, URDF)
Before this commit: robot upmoon, 15 links, 14 joints
Joints:
- joint wheel_lb_joint: axis 0 1 0 -> 0 -1 0
- joint wheel_lf_joint: axis 0 1 0 -> 0 -1 0
- joint wheel_lm_joint: axis 0 1 0 -> 0 -1 0

Commit message: Add limits to digging angle

File: upmoon_description/urdf/upmoon_description.urdf (robot description, URDF)
Before this commit: robot upmoon, 15 links, 14 joints
Links:
- added link dig_angle_link
Joints:
- added joint dig_angle_joint: type continuous, parent base_link, child dig_angle_link, axis 0 -1 0

Commit message: Add fake digging body to load model

File: upmoon_description/urdf/upmoon_description.urdf (robot description, URDF)
Before this commit: robot upmoon, 16 links, 15 joints
Links:
- link dig_angle_link: mass None -> 1; geometry visual cylinder length=0.01 radius=0.01

Commit message: Update model and joystick.

File: upmoon_description/urdf/upmoon_description.urdf (robot description, URDF)
Before this commit: robot upmoon, 16 links, 15 joints
Joints:
- joint ankle_lb_joint: axis 0 0 1 -> 0 0 -1
- joint ankle_rf_joint: axis 0 0 1 -> 0 0 -1
- joint ankle_rm_joint: axis 0 0 1 -> 0 0 -1

Commit message: Add starter code for actions to rotate a-joints while spinning the drive wheels.

File: upmoon_description/urdf/upmoon_description.urdf (robot description, URDF)
Before this commit: robot upmoon, 16 links, 15 joints
Joints:
- joint ankle_lb_joint: limit (none) -> lower=0 upper=3.1415 effort=27 velocity=0.8727
- joint ankle_lf_joint: limit (none) -> lower=0 upper=3.1415 effort=27 velocity=0.8727
- joint ankle_lm_joint: limit (none) -> lower=0 upper=3.1415 effort=27 velocity=0.8727
- joint ankle_rb_joint: limit (none) -> lower=0 upper=3.1415 effort=27 velocity=0.8727
- joint ankle_rf_joint: limit (none) -> lower=0 upper=3.1415 effort=27 velocity=0.8727
- joint ankle_rm_joint: limit (none) -> lower=0 upper=3.1415 effort=27 velocity=0.8727

Commit message: Control ankle joints by action server. Add dynamic reconfig to articulate action. Add interactive shell for teleop articulate client. Add deposition linear actuators.

File: upmoon_description/urdf/upmoon_description.urdf (robot description, URDF)
Before this commit: robot upmoon, 16 links, 15 joints
Links:
- added link dummy
- link dig_angle_link: geometry 
Joints:
- added joint dummy_joint: type fixed, parent dummy, child base_link

Commit message: update origin of f & b wheels

File: upmoon_description/urdf/upmoon_description.urdf (robot description, URDF)
Before this commit: robot upmoon, 17 links, 16 joints
Joints:
- joint ankle_lb_joint: limit lower=0 upper=3.1415 effort=27 velocity=0.8727 -> lower=1.57 upper=3.1415 effort=27 velocity=0.8727; origin xyz=-0.41873 0.18733 0.15178 rpy=0 0 0 -> xyz=-0.41873 0.18733 0.15178 rpy=0 0 1.57
- joint ankle_lf_joint: limit lower=0 upper=3.1415 effort=27 velocity=0.8727 -> lower=1.57 upper=3.1415 effort=27 velocity=0.8727; origin xyz=0.39333 0.18733 0.15178 rpy=0 0 0 -> xyz=0.39333 0.18733 0.15178 rpy=0 0 1.57
- joint ankle_rb_joint: limit lower=0 upper=3.1415 effort=27 velocity=0.8727 -> lower=1.57 upper=3.1415 effort=27 velocity=0.8727; origin xyz=-0.41873 -0.18733 0.15178 rpy=0 0 0 -> xyz=-0.41873 -0.18733 0.15178 rpy=0 0 1.57
- joint ankle_rf_joint: limit lower=0 upper=3.1415 effort=27 velocity=0.8727 -> lower=1.57 upper=3.1415 effort=27 velocity=0.8727; origin xyz=0.39333 -0.18733 0.15178 rpy=0 0 0 -> xyz=0.39333 -0.18733 0.15178 rpy=0 0 1.57

Commit message: Fix ankles to only turn 90 degrees.

File: upmoon_description/urdf/upmoon_description.urdf (robot description, URDF)
Before this commit: robot upmoon, 17 links, 16 joints
Joints:
- joint ankle_lb_joint: origin xyz=-0.41873 0.18733 0.15178 rpy=0 0 1.57 -> xyz=-0.41873 0.18733 0.15178 rpy=0 0 -1.57
- joint ankle_rf_joint: origin xyz=0.39333 -0.18733 0.15178 rpy=0 0 1.57 -> xyz=0.39333 -0.18733 0.15178 rpy=0 0 -1.57

Commit message: changing software to match mechanical changes in wheel position

File: upmoon_description/urdf/upmoon_description.urdf (robot description, URDF)
Before this commit: robot upmoon, 17 links, 16 joints
Joints:
- joint ankle_lb_joint: origin xyz=-0.41873 0.18733 0.15178 rpy=0 0 -1.57 -> xyz=-0.41873 0.18733 0.15178 rpy=0 0 -3.14
- joint ankle_lf_joint: origin xyz=0.39333 0.18733 0.15178 rpy=0 0 1.57 -> xyz=0.39333 0.18733 0.15178 rpy=0 0 3.14
- joint ankle_lm_joint: origin xyz=-0.035934 0.18733 0.15178 rpy=0 0 0 -> xyz=-0.035934 0.18733 0.15178 rpy=0 0 3.14; type continuous -> fixed
- joint ankle_rb_joint: origin xyz=-0.41873 -0.18733 0.15178 rpy=0 0 1.57 -> xyz=-0.41873 -0.18733 0.15178 rpy=0 0 3.14
- joint ankle_rf_joint: origin xyz=0.39333 -0.18733 0.15178 rpy=0 0 -1.57 -> xyz=0.39333 -0.18733 0.15178 rpy=0 0 -3.14
- joint ankle_rm_joint: origin xyz=-0.035934 -0.18733 0.15178 rpy=0 0 0 -> xyz=-0.035934 -0.18733 0.15178 rpy=0 0 -3.14; type continuous -> fixed
